File: hardware/board/radicon-client/radicon-client.kicad_pcb (KiCad board)
At the start: 2 copper layers, 24 x 84 mm, 7 parts, among them J1 PIN, Q1 NMOS, U1 TWE-L-DP-W

Commit message: update board
Parts:
- added SW1: SW_DIP_x01, Jumper:SolderJumper-2_P1.3mm_Open_TrianglePad1.0x1.5mm, F.Cu at (146.3, 91.9)
- added SW2: SW_DIP_x01, Jumper:SolderJumper-2_P1.3mm_Open_TrianglePad1.0x1.5mm, F.Cu at (143.4, 91.9)
- added SW3: SW_DIP_x01, Jumper:SolderJumper-2_P1.3mm_Open_TrianglePad1.0x1.5mm, F.Cu at (140.4, 91.9)
- J1: moved to B.Cu
- moved R1 3.80 mm to (139.7, 73.2)
- moved Q1 3.01 mm to (145.5, 77.2), turned to 90 degrees
- moved J1 2.50 mm to (143.0, 69.5), turned to 0 degrees
- moved BT1 1.25 mm to (144.0, 116.0)
Connections:
- U1 pad 13: unconnected-(U1-DIO10/M1-Pad13) -> Net-(U1-DIO10/M1)
- U1 pad 26: unconnected-(U1-DIO2/M2-Pad26) -> Net-(U1-DIO2/M2)
- U1 pad 27: unconnected-(U1-DIO3/M3-Pad27) -> Net-(U1-DIO3/M3)
Routing:
- net Net-(U1-DIO10/M1): track 0.00 -> 42.8 mm, vias 0 -> 1
- net GND: track 1.30 -> 25.4 mm, vias 1 -> 0
- net Net-(U1-DIO2/M2): track 0.00 -> 11.2 mm, vias 0 -> 1
- net Net-(J1-Pin_1): track 4.76 -> 15.4 mm, vias 0 -> 1
- net Net-(U1-DIO3/M3): track 0.00 -> 6.86 mm
- net Net-(Q1-G): track 25.8 -> 31.1 mm
- net +3V0: track 28.9 -> 29.6 mm
